Commit message: ...

File: src/fwsbot/description/urdf/fwsbot.core.xacro (robot description, xacro)
@@ -2,6 +2,6 @@
 <robot xmlns:xacro="http://ros.org/wiki/xacro">
   <!-- ============= Materials & Intertias =============  -->
-  <xacro:include filename="$(find fws_description)/urdf/inertial_macros.xacro"/>
-  <xacro:include filename="$(find fws_description)/urdf/materials.xacro"/>
+  <xacro:include filename="$(find fwsbot)/urdf/inertial_macros.xacro"/>
+  <xacro:include filename="$(find fwsbot)/urdf/materials.xacro"/>
   <!-- =============== Links & Joints =============== -->
   <!-- Base  footprint-->
@@ -25,5 +25,5 @@
       <geometry>
         <!-- <box size="0.90 0.72 0.15"/> -->
-        <mesh filename="package://fws_description/meshes/base_link.stl" scale="0.001 0.001 0.001" />
+        <mesh filename="package://fwsbot/meshes/base_link.stl" scale="0.001 0.001 0.001" />
       </geometry>
       <material name="blue"/>
@@ -51,5 +51,5 @@
       <geometry>
         <box size="0.07 0.07 0.15"/>
-        <!-- <mesh filename="package://fws_description/meshes/steering_link.stl" scale="0.001 0.001 0.001"/> -->
+        <!-- <mesh filename="package://fwsbot/meshes/steering_link.stl" scale="0.001 0.001 0.001"/> -->
       </geometry>
       <material name="grey"/>
@@ -77,5 +77,5 @@
       <geometry>
         <box size="0.07 0.07 0.15"/>
-        <!-- <mesh filename="package://fws_description/meshes/steering_link.stl" scale="0.001 0.001 0.001"/> -->
+        <!-- <mesh filename="package://fwsbot/meshes/steering_link.stl" scale="0.001 0.001 0.001"/> -->
       </geometry>
       <material name="grey"/>
@@ -103,5 +103,5 @@
       <geometry>
         <box size="0.07 0.07 0.15"/>
-        <!-- <mesh filename="package://fws_description/meshes/steering_link.stl" scale="0.001 0.001 0.001"/> -->
+        <!-- <mesh filename="package://fwsbot/meshes/steering_link.stl" scale="0.001 0.001 0.001"/> -->
       </geometry>
       <material name="grey"/>
@@ -129,5 +129,5 @@
       <geometry>
         <box size="0.07 0.07 0.15"/>
-        <!-- <mesh filename="package://fws_description/meshes/steering_link.stl" scale="0.001 0.001 0.001"/> -->
+        <!-- <mesh filename="package://fwsbot/meshes/steering_link.stl" scale="0.001 0.001 0.001"/> -->
       </geometry>
       <material name="grey"/>
@@ -154,5 +154,5 @@
       <geometry>
         <cylinder radius="0.13" length="0.08"/>
-        <!-- <mesh filename="package://fws_description/meshes/wheel.stl" scale="0.001 0.001 0.001"/> -->
+        <!-- <mesh filename="package://fwsbot/meshes/wheel.stl" scale="0.001 0.001 0.001"/> -->
       </geometry>
       <material name="green"/>
@@ -180,5 +180,5 @@
       <geometry>
         <cylinder radius="0.13" length="0.08"/>
-       <!-- <mesh filename="package://fws_description/meshes/wheel.stl" scale="0.001 0.001 0.001"/> -->
+       <!-- <mesh filename="package://fwsbot/meshes/wheel.stl" scale="0.001 0.001 0.001"/> -->
       </geometry>
       <material name="green"/>
@@ -206,5 +206,5 @@
       <geometry>
         <cylinder radius="0.13" length="0.08"/>
-        <!-- <mesh filename="package://fws_description/meshes/wheel.stl" scale="0.001 0.001 0.001"/> -->
+        <!-- <mesh filename="package://fwsbot/meshes/wheel.stl" scale="0.001 0.001 0.001"/> -->
       </geometry>
       <material name="green"/>
@@ -232,5 +232,5 @@
       <geometry>
         <cylinder radius="0.13" length="0.08"/>
-        <!-- <mesh filename="package://fws_description/meshes/wheel.stl" scale="0.001 0.001 0.001"/> -->
+        <!-- <mesh filename="package://fwsbot/meshes/wheel.stl" scale="0.001 0.001 0.001"/> -->
       </geometry>
       <material name="green"/>
